File: PCB_Files/bluepill.kicad_pcb (KiCad board)
At the start: 2 copper layers, 21.3 x 53.3 mm, 7 parts, among them J1 TYPE-C-31-M12_13, J2 Conn_01x20_Female, J3 Conn_01x20_Female, J4 Conn_01x06_Female, J5 Conn_01x04_Female, SW1 SW_Push, U1 STM32F103x8_B-LQFP48

Commit message: Further tracing
Parts:
- added C1: 100n, Capacitor_SMD:C_0402_1005Metric, F.Cu at (145.3, 93.7)
- added C2: 100n, Capacitor_SMD:C_0402_1005Metric, F.Cu at (118.0, 95.8)
- added C3: 100n, Capacitor_SMD:C_0402_1005Metric, F.Cu at (122.8, 95.0)
- added C4: 1u, Capacitor_SMD:C_0402_1005Metric, F.Cu at (125.7, 95.0)
- added C5: 10u, Capacitor_SMD:C_0402_1005Metric, F.Cu at (120.9, 97.0)
- added C6: 100n, Capacitor_SMD:C_0402_1005Metric, F.Cu at (123.8, 97.0)
- added D1: D_Schottky_Small, Diode_SMD:D_0603_1608Metric, B.Cu at (150.1, 80.1)
- added F1: 0.5A trip, Fuse:Fuse_0603_1608Metric, B.Cu at (150.1, 78.5)
- added Q1: DTC143Z, Package_TO_SOT_SMD:SOT-23, B.Cu at (145.7, 119.0)
- added R1: 22R, Resistor_SMD:R_0402_1005Metric, B.Cu at (149.2, 87.0)
- added R2: 22R, Resistor_SMD:R_0402_1005Metric, B.Cu at (148.1, 87.0)
- added R3: 100k, Resistor_SMD:R_0402_1005Metric, B.Cu at (151.0, 93.7)
- added R4: 100k, Resistor_SMD:R_0402_1005Metric, B.Cu at (153.3, 93.7)
- added R5: 10k, Resistor_SMD:R_0402_1005Metric, F.Cu at (147.3, 93.7)
- added R6: 1R, Resistor_SMD:R_0402_1005Metric, B.Cu at (146.9, 116.6)
- added R7: 100k, Resistor_SMD:R_0402_1005Metric, F.Cu at (126.7, 97.0)
- added R8: 1k, Resistor_SMD:R_0402_1005Metric, B.Cu at (144.9, 116.6)
- added U3: TPS709xxDBV, acheron_Components:SOT-23-5, B.Cu at (145.4, 87.0)
- added U4: USBLC6-2SC6, acheron_Components:SOT-23-6, B.Cu at (145.3, 93.2)
- U1: footprint acheron_Components:LQFP-48_7x7mm_P0.5mm -> acheron_Components:UQFN-48-1EP_6x6mm_P0.4mm_EP4.62x4.62mm
- moved SW1 0.25 mm to (146.3, 88.9)
Connections:
- net Net-(J3-Pad8) renamed PA11
- net Net-(J3-Pad9) renamed PA12
- net Net-(J5-Pad2) renamed SWD
- net Net-(J5-Pad3) renamed SWDIO
- net Net-(U1-Pad34) renamed PA13
- net Net-(U1-Pad37) renamed SWCLK
- J1 pad A4: Net-(J1-PadA4) -> VBUS
- J1 pad A6: Net-(J1-PadA6) -> /ConnUSBP
- J1 pad A7: Net-(J1-PadA7) -> /ConnUSBN
- J1 pad B4: Net-(J1-PadB4) -> VBUS
- J1 pad B6: Net-(J1-PadB6) -> /ConnUSBP
- J1 pad B7: Net-(J1-PadB7) -> /ConnUSBN
- J2 pad 1: Net-(J2-Pad1) -> GND
- J2 pad 10: Net-(J2-Pad10) -> PA6
- J2 pad 11: Net-(J2-Pad11) -> PA5
- J2 pad 12: Net-(J2-Pad12) -> PA4
- J2 pad 13: Net-(J2-Pad13) -> PA3
- J2 pad 14: Net-(J2-Pad14) -> PA2
- J2 pad 15: Net-(J2-Pad15) -> PA1
- J2 pad 16: Net-(J2-Pad16) -> PA0
- J2 pad 17: Net-(J2-Pad17) -> PC15
- J2 pad 18: Net-(J2-Pad18) -> PC14
- J2 pad 19: GND -> PC13
- J2 pad 2: Net-(J2-Pad2) -> GND
- J2 pad 20: Net-(J2-Pad20) -> VBAT
- J2 pad 3: Net-(J2-Pad3) -> 3V3
- J2 pad 4: Net-(J2-Pad4) -> RST
- J2 pad 5: Net-(J2-Pad5) -> PB11
- J2 pad 6: Net-(J2-Pad6) -> PB10
- J2 pad 7: Net-(J2-Pad7) -> PB1
- J2 pad 8: Net-(J2-Pad8) -> PB0
- J2 pad 9: Net-(J2-Pad9) -> PA7
- J3 pad 1: GND -> PB12
- J3 pad 10: Net-(J3-Pad10) -> PA15
- J3 pad 11: Net-(J3-Pad11) -> PB3
- J3 pad 12: Net-(J3-Pad12) -> PB4
- J3 pad 13: Net-(J3-Pad13) -> PB5
- J3 pad 14: Net-(J3-Pad14) -> PB6
- J3 pad 15: Net-(J3-Pad15) -> PB7
- J3 pad 16: Net-(J3-Pad16) -> PB8
- J3 pad 17: Net-(J3-Pad17) -> PB9
- J3 pad 18: Net-(J3-Pad18) -> 5V
- J3 pad 19: Net-(J3-Pad19) -> GND
- J3 pad 2: GND -> PB13
- J3 pad 20: Net-(J3-Pad20) -> 3V3
- J3 pad 3: Net-(J3-Pad3) -> PB14
- J3 pad 4: Net-(J3-Pad4) -> PB15
- J3 pad 5: Net-(J3-Pad5) -> PA8
- J3 pad 6: Net-(J3-Pad6) -> PA9
- J3 pad 7: Net-(J3-Pad7) -> PA10
- J4 pad 1: Net-(J4-Pad1) -> 3V3
- J4 pad 3: Net-(J4-Pad3) -> GND
- J4 pad 4: Net-(J4-Pad4) -> GND
- J4 pad 6: Net-(J4-Pad6) -> 3V3
- J5 pad 1: Net-(J5-Pad1) -> JTAG_3V3
- SW1 pad 1: Net-(SW1-Pad1) -> GND
- SW1 pad 2: Net-(SW1-Pad2) -> RST
- U1 pad 1: Net-(U1-Pad1) -> VBAT
- U1 pad 10: Net-(U1-Pad10) -> PA0
- U1 pad 11: Net-(U1-Pad11) -> PA1
- U1 pad 12: Net-(U1-Pad12) -> PA2
- U1 pad 13: Net-(U1-Pad13) -> PA3
- U1 pad 14: Net-(U1-Pad14) -> PA4
- U1 pad 15: Net-(U1-Pad15) -> PA5
- U1 pad 16: Net-(U1-Pad16) -> PA6
- U1 pad 17: Net-(U1-Pad17) -> PA7
- U1 pad 18: Net-(U1-Pad18) -> PB0
- U1 pad 19: Net-(U1-Pad19) -> PB1
- U1 pad 2: Net-(U1-Pad2) -> PC13
- U1 pad 20: Net-(U1-Pad20) -> BOOT1
- U1 pad 21: Net-(U1-Pad21) -> PB10
- U1 pad 22: Net-(U1-Pad22) -> PB11
- U1 pad 25: Net-(U1-Pad25) -> PB12
- U1 pad 26: Net-(U1-Pad26) -> PB13
- U1 pad 27: Net-(U1-Pad27) -> PB14
- U1 pad 28: Net-(U1-Pad28) -> PB15
- U1 pad 29: Net-(U1-Pad29) -> PA8
- U1 pad 3: Net-(U1-Pad3) -> PC14
- U1 pad 30: Net-(U1-Pad30) -> PA9
- U1 pad 31: Net-(U1-Pad31) -> PA10
- U1 pad 32: Net-(U1-Pad32) -> DN
- U1 pad 33: Net-(U1-Pad33) -> DP
- U1 pad 35: Net-(U1-Pad35) -> GND
- U1 pad 38: Net-(U1-Pad38) -> PA15
- U1 pad 39: Net-(U1-Pad39) -> PB3
- U1 pad 4: Net-(U1-Pad4) -> PC15
- U1 pad 40: Net-(U1-Pad40) -> PB4
- U1 pad 41: Net-(U1-Pad41) -> PB5
- U1 pad 42: Net-(U1-Pad42) -> PB6
- U1 pad 43: Net-(U1-Pad43) -> PB7
- U1 pad 44: Net-(U1-Pad44) -> BOOT0
- U1 pad 45: Net-(U1-Pad45) -> PB8
- U1 pad 46: Net-(U1-Pad46) -> PB9
- U1 pad 47: Net-(U1-Pad47) -> GND
- U1 pad 7: Net-(U1-Pad7) -> RST
- U1 pad 8: Net-(U1-Pad8) -> GND
Routing:
- net 3V3: track 0.00 -> 49.3 mm, vias 0 -> 1
- net LDO_EN: track 0.00 -> 35.2 mm
- net PB12: track 0.00 -> 25.6 mm
- net PB15: track 0.00 -> 25.3 mm, vias 0 -> 1
- net VBAT: track 0.00 -> 24.1 mm
- net PB13: track 0.00 -> 23.6 mm
- net PB14: track 0.00 -> 23.0 mm
- net PC13: track 0.00 -> 22.0 mm
- net RST: track 0.00 -> 21.7 mm
- net PA8: track 0.00 -> 21.1 mm, vias 0 -> 1
- net PC14: track 0.00 -> 19.9 mm
- net PA9: track 0.00 -> 18.2 mm, vias 0 -> 1
- net PC15: track 0.00 -> 17.8 mm
- net PA0: track 0.00 -> 17.6 mm
- net PA10: track 0.00 -> 17.5 mm, vias 0 -> 1
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Other:
- net class Default: clearance 0.2 -> 0.127; trace_width 0.25 -> 0.254
- rule trace_clearance: 0.2 -> 0.127

Commit message: Further routing
Parts:
- removed Q1: DTC143Z, Package_TO_SOT_SMD:SOT-23
- added C7: 4.7n, Capacitor_SMD:C_0402_1005Metric, F.Cu at (157.5, 77.1)
- added C8: 12p, Capacitor_SMD:C_0402_1005Metric, B.Cu at (154.1, 107.6)
- added C9: 12p, Capacitor_SMD:C_0402_1005Metric, B.Cu at (155.3, 107.5)
- added RCC1: 5.1k, Resistor_SMD:R_0402_1005Metric, F.Cu at (154.4, 84.7)
- added RCC2: 5.1k, Resistor_SMD:R_0402_1005Metric, F.Cu at (144.3, 82.8)
- added Y1: 16MHz, Crystal:Crystal_SMD_2016-4Pin_2.0x1.6mm, B.Cu at (154.6, 110.0)
- C2: value 100n -> 1u; moved to B.Cu
- C3: value 100n -> 10u; moved to B.Cu
- C4, C5, C6: moved to B.Cu
- F1: value 0.5A trip -> 1.0A trip
- R6: value 1R -> 1M; moved to F.Cu
- R8: value 1k -> 330R; moved to F.Cu
- moved R6 40.0 mm to (155.8, 77.6), turned to 270 degrees
- moved C2 38.1 mm to (146.6, 120.9), turned to 180 degrees
- moved C5 32.4 mm to (149.4, 81.7)
- moved R7 31.0 mm to (146.5, 120.9)
- moved C4 26.4 mm to (147.2, 79.6), turned to 180 degrees
- moved C3 25.5 mm to (146.2, 84.7)
- moved C6 25.4 mm to (148.5, 91.1), turned to 180 degrees
- moved R8 23.1 mm to (147.2, 93.6)
- moved C1 2.10 mm to (147.2, 94.6)
- moved R5 1.91 mm to (147.2, 95.6)
- moved F1 0.50 mm to (149.7, 78.8)
- moved D1 0.46 mm to (149.7, 80.4)
- moved J1 0.25 mm to (149.9, 83.1)
Connections:
- J1 pad S: Net-(J1-PadS) -> Net-(C7-Pad2)
- J5 pad 1: JTAG_3V3 -> 3V3
- R6 pad 1: JTAG_3V3 -> Net-(C7-Pad2)
- R6 pad 2: 3V3 -> GND
- R8 pad 1: LDO_EN -> RST
- R8 pad 2: 3V3 -> Net-(R8-Pad2)
- SW1 pad 2: RST -> Net-(R8-Pad2)
- U3 pad 5: LDO_EN -> 5V
Routing:
- net 5V: track 4.29 -> 56.0 mm
- net 3V3: track 49.3 -> 86.3 mm
- net LDO_EN: track 35.2 -> 0.00 mm
- net Net-(C7-Pad2): track 0.00 -> 20.7 mm
- net PB9: track 0.00 -> 20.6 mm
- net PB8: track 0.00 -> 18.7 mm
- net Net-(J1-PadS): track 17.0 -> 0.00 mm
- net RST: track 21.7 -> 37.3 mm, vias 0 -> 1
- net PA15: track 0.00 -> 15.5 mm
- net VBUS: track 15.4 -> 30.8 mm
- net PB7: track 0.00 -> 15.1 mm
- net PA2: track 0.00 -> 14.0 mm
- net PB6: track 0.00 -> 12.3 mm
- net Net-(C9-Pad1): track 0.00 -> 12.3 mm, vias 0 -> 1
- net PB3: track 0.00 -> 9.99 mm
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Other:
- board text added: "Acheron BluePill"
- board text added: "AcheronProject"
- board text added: "V. 0.1"
